Commit message: Add motor display

File: mrobot_description/urdf/mrobot.urdf.xacro (robot description, xacro)
@@ -1,5 +1,10 @@
 <?xml version="1.0"?>
 <robot name="mrobot" xmlns:xacro="http://ros.org/wiki/xacro">
+  <xacro:include filename="$(find mrobot_description)/urdf/common_properties.xacro"/>
   <xacro:property name="wheel_radius" value="0.033"/>
+  <xacro:property name="motor_radius" value="0.02"/>
+  <xacro:property name="motor_length" value="0.08"/>
+  <xacro:property name="motor_x" value="-0.055"/>
+  <xacro:property name="motor_y_dist" value="0.150"/>
   <link name="base_footprint"/>
   <link name="base_link">
@@ -10,3 +15,22 @@
     <child link="base_link" />
   </joint>
+  <xacro:macro name="motor" params="prefix yreflect">
+    <link name="${prefix}_motor">
+      <visual>
+        <origin xyz="0 0 0" rpy="${pi/2} 0 0" />
+        <geometry>
+          <cylinder radius="${motor_radius}" length="${motor_length}"/>
+        </geometry>
+        <origin rpy="0 0 0" xyz="0 0 0"/>
+        <material name="gray" />
+      </visual>
+    </link>
+    <joint name="base_${prefix}_motor_joint" type="fixed">
+      <origin xyz="${motor_x} ${motor_y_dist/2*yreflect} 0" rpy="0 0 0" />
+      <parent link="base_link"/>
+      <child link="${prefix}_motor" />
+    </joint>
+  </xacro:macro>
+  <xacro:motor prefix="left" yreflect="1"/>
+  <xacro:motor prefix="right" yreflect="-1"/>
 </robot>

Commit message: Add wheel display

File: mrobot_description/urdf/mrobot.urdf.xacro (robot description, xacro)
@@ -3,4 +3,5 @@
   <xacro:include filename="$(find mrobot_description)/urdf/common_properties.xacro"/>
   <xacro:property name="wheel_radius" value="0.033"/>
+  <xacro:property name="wheel_length" value="0.017"/>
   <xacro:property name="motor_radius" value="0.02"/>
   <xacro:property name="motor_length" value="0.08"/>
@@ -32,5 +33,23 @@
     </joint>
   </xacro:macro>
-  <xacro:motor prefix="left" yreflect="1"/>
-  <xacro:motor prefix="right" yreflect="-1"/>
+  <xacro:macro name="wheel" params="prefix yreflect">
+    <xacro:motor prefix="${prefix}" yreflect="${yreflect}"/>
+    <link name="${prefix}_wheel_link">
+      <visual>
+        <geometry>
+          <cylinder radius="${wheel_radius}" length="${wheel_length}"/>
+        </geometry>
+        <origin xyz="0 0 0" rpy="${pi/2} 0 0"/>
+        <material name="white" />
+      </visual>
+    </link>
+    <joint name="${prefix}_wheel_joint" type="continuous">
+      <origin xyz="0 ${(motor_length+wheel_length)/2*yreflect} 0" rpy="0 0 0"/>
+      <parent link="${prefix}_motor"/>
+      <child link="${prefix}_wheel_link"/>
+      <axis xyz="0 1 0"/>
+    </joint>
+  </xacro:macro>
+  <xacro:wheel prefix="left" yreflect="1"/>
+  <xacro:wheel prefix="right" yreflect="-1"/>
 </robot>

Commit message: Add caster display

File: mrobot_description/urdf/mrobot.urdf.xacro (robot description, xacro)
@@ -4,4 +4,6 @@
   <xacro:property name="wheel_radius" value="0.033"/>
   <xacro:property name="wheel_length" value="0.017"/>
+  <xacro:property name="base_link_radius" value="0.13"/>
+  <xacro:property name="base_link_length" value="0.005"/>
   <xacro:property name="motor_radius" value="0.02"/>
   <xacro:property name="motor_length" value="0.08"/>
@@ -53,3 +55,17 @@
   <xacro:wheel prefix="left" yreflect="1"/>
   <xacro:wheel prefix="right" yreflect="-1"/>
+  <link name="front_caster_link">
+    <visual>
+      <geometry>
+        <sphere radius="${wheel_radius/2}" />
+      </geometry>
+      <origin xyz="0 0 0" rpy="${pi/2} 0 0"/>
+      <material name="black" />
+    </visual>
+  </link>
+  <joint name="front_caster_joint" type="fixed">
+    <origin xyz="${base_link_radius-wheel_radius/2} 0 -${wheel_radius/2}" rpy="0 0 0"/>
+    <parent link="base_link"/>
+    <child link="front_caster_link"/>
+  </joint>
 </robot>

Commit message: Add plate1 display

File: mrobot_description/urdf/mrobot.urdf.xacro (robot description, xacro)
@@ -10,4 +10,5 @@
   <xacro:property name="motor_x" value="-0.055"/>
   <xacro:property name="motor_y_dist" value="0.150"/>
+  <xacro:property name="plate_height" value="0.07"/>
   <link name="base_footprint"/>
   <link name="base_link">
@@ -69,3 +70,17 @@
     <child link="front_caster_link"/>
   </joint>
+  <link name="plate_1_link">
+    <visual>
+      <geometry>
+        <cylinder radius="${base_link_radius}" length="${base_link_length}"/>
+      </geometry>
+      <origin xyz=" 0 0 0 " rpy="0 0 0" />
+      <material name="yellow"/>
+    </visual>
+  </link>
+  <joint name="plate_1_joint" type="fixed">
+    <origin xyz="0 0 ${plate_height}" rpy="0 0 0" />
+    <parent link="base_link"/>
+    <child link="plate_1_link"/>
+  </joint>
 </robot>

Commit message: Add base_link display

File: mrobot_description/urdf/mrobot.urdf.xacro (robot description, xacro)
@@ -13,4 +13,11 @@
   <link name="base_footprint"/>
   <link name="base_link">
+    <visual>
+      <geometry>
+        <cylinder radius="${base_link_radius}" length="${base_link_length}"/>
+      </geometry>
+      <origin xyz=" 0 0 0" rpy="0 0 0" />
+      <material name="yellow" />
+    </visual>
   </link>
   <joint name="base_footprint_joint" type="fixed">

Commit message: Add colliders for some objects

File: mrobot_description/urdf/mrobot.urdf.xacro (robot description, xacro)
@@ -20,4 +20,10 @@
       <material name="yellow" />
     </visual>
+    <collision>
+      <geometry>
+        <cylinder radius="${base_link_radius}" length="${base_link_length}"/>
+      </geometry>
+      <origin xyz=" 0 0 0" rpy="0 0 0" />
+    </collision>
   </link>
   <joint name="base_footprint_joint" type="fixed">
@@ -36,4 +42,10 @@
         <material name="gray" />
       </visual>
+      <collision>
+        <geometry>
+          <cylinder radius="${motor_radius}" length="${motor_length}"/>
+        </geometry>
+        <origin xyz="0 0 0" rpy="${pi/2} 0 0" />
+      </collision>
     </link>
     <joint name="base_${prefix}_motor_joint" type="fixed">
@@ -53,4 +65,10 @@
         <material name="white" />
       </visual>
+      <collision>
+        <geometry>
+          <cylinder radius="${wheel_radius}" length="${wheel_length}"/>
+        </geometry>
+        <origin xyz="0 0 0" rpy="${pi/2} 0 0"/>
+      </collision>
     </link>
     <joint name="${prefix}_wheel_joint" type="continuous">
@@ -71,4 +89,10 @@
       <material name="black" />
     </visual>
+    <collision>
+      <geometry>
+        <sphere radius="${wheel_radius/2}" />
+      </geometry>
+      <origin xyz="0 0 0.01" rpy="${pi/2} 0 0"/>
+    </collision>
   </link>
   <joint name="front_caster_joint" type="fixed">

Commit message: Fix a bug

File: mrobot_description/urdf/mrobot.urdf.xacro (robot description, xacro)
@@ -35,9 +35,8 @@
     <link name="${prefix}_motor">
       <visual>
-        <origin xyz="0 0 0" rpy="${pi/2} 0 0" />
         <geometry>
           <cylinder radius="${motor_radius}" length="${motor_length}"/>
         </geometry>
-        <origin rpy="0 0 0" xyz="0 0 0"/>
+        <origin xyz="0 0 0" rpy="${pi/2} 0 0" />
         <material name="gray" />
       </visual>

Commit message: Add inertia matrix properites to some objects

File: mrobot_description/urdf/mrobot.urdf.xacro (robot description, xacro)
@@ -26,4 +26,11 @@
       <origin xyz=" 0 0 0" rpy="0 0 0" />
     </collision>
+    <inertial>
+      <origin xyz="0 0 0" />
+      <mass value="2" />
+      <inertia ixx="0.001" ixy="0.0" ixz="0.0"
+               iyy="0.001" iyz="0.0"
+               izz="0.5" />
+    </inertial>
   </link>
   <joint name="base_footprint_joint" type="fixed">
@@ -47,4 +54,11 @@
         <origin xyz="0 0 0" rpy="${pi/2} 0 0" />
       </collision>
+      <inertial>
+        <origin xyz="0 0 0" />
+        <mass value="0.1" />
+        <inertia ixx="0.001" ixy="0.0" ixz="0.0"
+          iyy="0.001" iyz="0.0"
+          izz="0.001" />
+      </inertial>
     </link>
     <joint name="base_${prefix}_motor_joint" type="fixed">
@@ -70,4 +84,11 @@
         <origin xyz="0 0 0" rpy="${pi/2} 0 0"/>
       </collision>
+      <inertial>
+        <origin xyz="0 0 0" />
+        <mass value="0.01" />
+        <inertia ixx="0.001" ixy="0.0" ixz="0.0"
+          iyy="0.001" iyz="0.0"
+          izz="0.001" />
+      </inertial>
     </link>
     <joint name="${prefix}_wheel_joint" type="continuous">
@@ -94,4 +115,11 @@
       <origin xyz="0 0 0.01" rpy="${pi/2} 0 0"/>
     </collision>
+    <inertial>
+      <origin xyz="0 0 0" />
+      <mass value="0.001" />
+      <inertia ixx="0.0001" ixy="0.0" ixz="0.0"
+        iyy="0.0001" iyz="0.0"
+        izz="0.0001" />
+    </inertial>
   </link>
   <joint name="front_caster_joint" type="fixed">

Commit message: Add support columns

File: mrobot_description/urdf/mrobot.urdf.xacro (robot description, xacro)
@@ -11,4 +11,6 @@
   <xacro:property name="motor_y_dist" value="0.150"/>
   <xacro:property name="plate_height" value="0.07"/>
+  <xacro:property name="standoff_x" value="0.12"/>
+  <xacro:property name="standoff_y" value="0.10"/>
   <link name="base_footprint"/>
   <link name="base_link">
@@ -128,4 +130,39 @@
     <child link="front_caster_link"/>
   </joint>
+  <xacro:macro name="mrobot_standoff_2in" params="parent number x_loc y_loc z_loc">
+    <link name="standoff_2in_${number}_link">
+      <visual>
+        <geometry>
+          <box size="0.01 0.01 0.07" />
+        </geometry>
+        <origin xyz=" 0 0 0 " rpy="0 0 0" />
+        <material name="black2">
+          <color rgba="0.16 0.17 0.15 0.9"/>
+        </material>
+      </visual>
+      <collision>
+        <geometry>
+          <box size="0.01 0.01 0.07" />
+        </geometry>
+        <origin xyz=" 0 0 0 " rpy="0 0 0" />
+      </collision>
+      <inertial>
+        <origin xyz="0 0 0" />
+        <mass value="0.001" />
+        <inertia ixx="0.0001" ixy="0.0" ixz="0.0"
+                 iyy="0.0001" iyz="0.0"
+                 izz="0.0001" />
+      </inertial>
+    </link>
+    <joint name="standoff_2in_${number}_joint" type="fixed">
+      <origin xyz="${x_loc} ${y_loc} ${z_loc}" rpy="0 0 0" />
+      <parent link="${parent}"/>
+      <child link="standoff_2in_${number}_link" />
+    </joint>
+  </xacro:macro>
+  <xacro:mrobot_standoff_2in parent="base_link" number="1" x_loc="-${standoff_x/2 + 0.03}" y_loc="-${standoff_y - 0.03}" z_loc="${plate_height/2}"/>
+  <xacro:mrobot_standoff_2in parent="base_link" number="2" x_loc="-${standoff_x/2 + 0.03}" y_loc="${standoff_y - 0.03}" z_loc="${plate_height/2}"/>
+  <xacro:mrobot_standoff_2in parent="base_link" number="3" x_loc="${standoff_x/2}" y_loc="-${standoff_y}" z_loc="${plate_height/2}"/>
+  <xacro:mrobot_standoff_2in parent="base_link" number="4" x_loc="${standoff_x/2}" y_loc="${standoff_y}" z_loc="${plate_height/2}"/>
   <link name="plate_1_link">
     <visual>

Commit message: Complete the collision and inertia properties of plate1

File: mrobot_description/urdf/mrobot.urdf.xacro (robot description, xacro)
@@ -173,4 +173,17 @@
       <material name="yellow"/>
     </visual>
+    <collision>
+      <geometry>
+        <cylinder radius="${base_link_radius}" length="${base_link_length}"/>
+      </geometry>
+      <origin xyz="0 0 0" rpy="0 0 0" />
+    </collision>
+    <inertial>
+      <origin xyz="0 0 0" />
+      <mass value="0.1" />
+      <inertia ixx="0.01" ixy="0.0" ixz="0.0"
+               iyy="0.01" iyz="0.0"
+               izz="0.01" />
+    </inertial>
   </link>
   <joint name="plate_1_joint" type="fixed">

Commit message: Add plate2

File: mrobot_description/urdf/mrobot.urdf.xacro (robot description, xacro)
@@ -192,3 +192,34 @@
     <child link="plate_1_link"/>
   </joint>
+  <xacro:mrobot_standoff_2in parent="standoff_2in_1_link" number="5" x_loc="0" y_loc="0" z_loc="${plate_height}"/>
+  <xacro:mrobot_standoff_2in parent="standoff_2in_2_link" number="6" x_loc="0" y_loc="0" z_loc="${plate_height}"/>
+  <xacro:mrobot_standoff_2in parent="standoff_2in_3_link" number="7" x_loc="0" y_loc="0" z_loc="${plate_height}"/>
+  <xacro:mrobot_standoff_2in parent="standoff_2in_4_link" number="8" x_loc="0" y_loc="0" z_loc="${plate_height}"/>
+  <link name="plate_2_link">
+    <visual>
+      <geometry>
+        <cylinder radius="${base_link_radius}" length="${base_link_length}"/>
+      </geometry>
+      <origin xyz="0 0 0" rpy="0 0 0" />
+      <material name="yellow" />
+    </visual>
+    <collision>
+      <geometry>
+        <cylinder radius="${base_link_radius}" length="${base_link_length}"/>
+      </geometry>
+      <origin xyz="0 0 0" rpy="0 0 0" />
+    </collision>
+    <inertial>
+      <origin xyz="0 0 0" />
+      <mass value="0.1" />
+      <inertia ixx="0.01" ixy="0.0" ixz="0.0"
+               iyy="0.01" iyz="0.0"
+               izz="0.01" />
+    </inertial>
+  </link>
+  <joint name="plate_2_joint" type="fixed">
+    <origin xyz="0 0 ${plate_height}" rpy="0 0 0" />
+    <parent link="plate_1_link"/>
+    <child link="plate_2_link"/>
+  </joint>
 </robot>

Commit message: Remove motor link

File: mrobot_description/urdf/mrobot.urdf.xacro (robot description, xacro)
@@ -3,5 +3,5 @@
   <xacro:include filename="$(find mrobot_description)/urdf/common_properties.xacro"/>
   <xacro:property name="wheel_radius" value="0.033"/>
-  <xacro:property name="wheel_length" value="0.017"/>
+  <xacro:property name="wheel_height" value="0.017"/>
   <xacro:property name="base_link_radius" value="0.13"/>
   <xacro:property name="base_link_length" value="0.005"/>
@@ -41,39 +41,9 @@
     <child link="base_link" />
   </joint>
-  <xacro:macro name="motor" params="prefix yreflect">
-    <link name="${prefix}_motor">
-      <visual>
-        <geometry>
-          <cylinder radius="${motor_radius}" length="${motor_length}"/>
-        </geometry>
-        <origin xyz="0 0 0" rpy="${pi/2} 0 0" />
-        <material name="gray" />
-      </visual>
-      <collision>
-        <geometry>
-          <cylinder radius="${motor_radius}" length="${motor_length}"/>
-        </geometry>
-        <origin xyz="0 0 0" rpy="${pi/2} 0 0" />
-      </collision>
-      <inertial>
-        <origin xyz="0 0 0" />
-        <mass value="0.1" />
-        <inertia ixx="0.001" ixy="0.0" ixz="0.0"
-          iyy="0.001" iyz="0.0"
-          izz="0.001" />
-      </inertial>
-    </link>
-    <joint name="base_${prefix}_motor_joint" type="fixed">
-      <origin xyz="${motor_x} ${motor_y_dist/2*yreflect} 0" rpy="0 0 0" />
-      <parent link="base_link"/>
-      <child link="${prefix}_motor" />
-    </joint>
-  </xacro:macro>
   <xacro:macro name="wheel" params="prefix yreflect">
-    <xacro:motor prefix="${prefix}" yreflect="${yreflect}"/>
     <link name="${prefix}_wheel_link">
       <visual>
         <geometry>
-          <cylinder radius="${wheel_radius}" length="${wheel_length}"/>
+          <cylinder radius="${wheel_radius}" length="${wheel_height}"/>
         </geometry>
         <origin xyz="0 0 0" rpy="${pi/2} 0 0"/>
@@ -82,5 +52,5 @@
       <collision>
         <geometry>
-          <cylinder radius="${wheel_radius}" length="${wheel_length}"/>
+          <cylinder radius="${wheel_radius}" length="${wheel_height}"/>
         </geometry>
         <origin xyz="0 0 0" rpy="${pi/2} 0 0"/>
@@ -95,6 +65,6 @@
     </link>
     <joint name="${prefix}_wheel_joint" type="continuous">
-      <origin xyz="0 ${(motor_length+wheel_length)/2*yreflect} 0" rpy="0 0 0"/>
-      <parent link="${prefix}_motor"/>
+      <origin xyz="${motor_x} ${base_link_radius*yreflect} 0" rpy="0 0 0"/>
+      <parent link="base_link"/>
       <child link="${prefix}_wheel_link"/>
       <axis xyz="0 1 0"/>

Commit message: Adjust the wheel position

File: mrobot_description/urdf/mrobot.urdf.xacro (robot description, xacro)
@@ -8,5 +8,5 @@
   <xacro:property name="motor_radius" value="0.02"/>
   <xacro:property name="motor_length" value="0.08"/>
-  <xacro:property name="motor_x" value="-0.055"/>
+  <xacro:property name="motor_x" value="-0.05"/>
   <xacro:property name="motor_y_dist" value="0.150"/>
   <xacro:property name="plate_height" value="0.07"/>

Commit message: Add some mass parameters

File: mrobot_description/urdf/mrobot.urdf.xacro (robot description, xacro)
@@ -4,11 +4,14 @@
   <xacro:property name="wheel_radius" value="0.033"/>
   <xacro:property name="wheel_height" value="0.017"/>
+  <xacro:property name="wheel_mass"   value="0.1" />
   <xacro:property name="base_link_radius" value="0.13"/>
   <xacro:property name="base_link_length" value="0.005"/>
-  <xacro:property name="motor_radius" value="0.02"/>
-  <xacro:property name="motor_length" value="0.08"/>
+  <xacro:property name="base_mass"        value="0.5" />
   <xacro:property name="motor_x" value="-0.05"/>
-  <xacro:property name="motor_y_dist" value="0.150"/>
+  <xacro:property name="caster_radius"         value="0.016" />
+  <xacro:property name="caster_joint_origin_x" value="-0.12" />
+  <xacro:property name="caster_mass"           value="0.01" />
   <xacro:property name="plate_height" value="0.07"/>
+  <xacro:property name="plate_mass"   value="0.05"/>
   <xacro:property name="standoff_x" value="0.12"/>
   <xacro:property name="standoff_y" value="0.10"/>

Commit message: Re-write caster

File: mrobot_description/urdf/mrobot.urdf.xacro (robot description, xacro)
@@ -76,31 +76,34 @@
   <xacro:wheel prefix="left" yreflect="1"/>
   <xacro:wheel prefix="right" yreflect="-1"/>
-  <link name="front_caster_link">
-    <visual>
-      <geometry>
-        <sphere radius="${wheel_radius/2}" />
-      </geometry>
-      <origin xyz="0 0 0" rpy="${pi/2} 0 0"/>
-      <material name="black" />
-    </visual>
-    <collision>
-      <geometry>
-        <sphere radius="${wheel_radius/2}" />
-      </geometry>
-      <origin xyz="0 0 0.01" rpy="${pi/2} 0 0"/>
-    </collision>
-    <inertial>
-      <origin xyz="0 0 0" />
-      <mass value="0.001" />
-      <inertia ixx="0.0001" ixy="0.0" ixz="0.0"
-        iyy="0.0001" iyz="0.0"
-        izz="0.0001" />
-    </inertial>
-  </link>
-  <joint name="front_caster_joint" type="fixed">
-    <origin xyz="${base_link_radius-wheel_radius/2} 0 -${wheel_radius/2}" rpy="0 0 0"/>
-    <parent link="base_link"/>
-    <child link="front_caster_link"/>
-  </joint>
+  <xacro:macro name="caster" params="fb xreflect">
+    <link name="${fb}_caster_link">
+      <visual>
+        <geometry>
+          <sphere radius="${caster_radius}" />
+        </geometry>
+        <origin xyz="0 0 0" rpy="0 0 0"/>
+        <material name="black" />
+      </visual>
+      <collision>
+        <geometry>
+          <sphere radius="${caster_radius}" />
+        </geometry>
+        <origin xyz="0 0 0" rpy="0 0 0"/>
+      </collision>
+      <inertial>
+        <origin xyz="0 0 0" />
+        <mass value="0.001" />
+        <inertia ixx="0.0001" ixy="0.0" ixz="0.0"
+          iyy="0.0001" iyz="0.0"
+          izz="0.0001" />
+      </inertial>
+    </link>
+    <joint name="{fb}_caster_joint" type="fixed">
+      <origin xyz="${caster_joint_origin_x*xreflect} 0 ${-caster_radius}" rpy="0 0 0"/>
+      <parent link="base_link"/>
+      <child link="${fb}_caster_link"/>
+    </joint>
+  </xacro:macro>
+  <xacro:caster fb="front" xreflect="-1"/>
   <xacro:macro name="mrobot_standoff_2in" params="parent number x_loc y_loc z_loc">
     <link name="standoff_2in_${number}_link">

Commit message: Re-wirte plate

File: mrobot_description/urdf/mrobot.urdf.xacro (robot description, xacro)
@@ -137,65 +137,42 @@
     </joint>
   </xacro:macro>
+  <xacro:macro name="plate" params="num parent">
+    <link name="plate_${num}_link">
+      <visual>
+        <geometry>
+          <cylinder radius="${base_link_radius}" length="${base_link_length}"/>
+        </geometry>
+        <origin xyz="0 0 0" rpy="0 0 0" />
+        <material name="yellow"/>
+      </visual>
+      <collision>
+        <geometry>
+          <cylinder radius="${base_link_radius}" length="${base_link_length}"/>
+        </geometry>
+        <origin xyz="0 0 0" rpy="0 0 0" />
+      </collision>
+      <inertial>
+        <origin xyz="0 0 0" />
+        <mass value="0.1" />
+        <inertia ixx="0.01" ixy="0.0" ixz="0.0"
+          iyy="0.01" iyz="0.0"
+          izz="0.01" />
+      </inertial>
+    </link>
+    <joint name="plate_${num}_joint" type="fixed">
+      <origin xyz="0 0 ${plate_height}" rpy="0 0 0" />
+      <parent link="${parent}"/>
+      <child link="plate_${num}_link"/>
+    </joint>
+  </xacro:macro>
   <xacro:mrobot_standoff_2in parent="base_link" number="1" x_loc="-${standoff_x/2 + 0.03}" y_loc="-${standoff_y - 0.03}" z_loc="${plate_height/2}"/>
   <xacro:mrobot_standoff_2in parent="base_link" number="2" x_loc="-${standoff_x/2 + 0.03}" y_loc="${standoff_y - 0.03}" z_loc="${plate_height/2}"/>
   <xacro:mrobot_standoff_2in parent="base_link" number="3" x_loc="${standoff_x/2}" y_loc="-${standoff_y}" z_loc="${plate_height/2}"/>
   <xacro:mrobot_standoff_2in parent="base_link" number="4" x_loc="${standoff_x/2}" y_loc="${standoff_y}" z_loc="${plate_height/2}"/>
-  <link name="plate_1_link">
-    <visual>
-      <geometry>
-        <cylinder radius="${base_link_radius}" length="${base_link_length}"/>
-      </geometry>
-      <origin xyz=" 0 0 0 " rpy="0 0 0" />
-      <material name="yellow"/>
-    </visual>
-    <collision>
-      <geometry>
-        <cylinder radius="${base_link_radius}" length="${base_link_length}"/>
-      </geometry>
-      <origin xyz="0 0 0" rpy="0 0 0" />
-    </collision>
-    <inertial>
-      <origin xyz="0 0 0" />
-      <mass value="0.1" />
-      <inertia ixx="0.01" ixy="0.0" ixz="0.0"
-               iyy="0.01" iyz="0.0"
-               izz="0.01" />
-    </inertial>
-  </link>
-  <joint name="plate_1_joint" type="fixed">
-    <origin xyz="0 0 ${plate_height}" rpy="0 0 0" />
-    <parent link="base_link"/>
-    <child link="plate_1_link"/>
-  </joint>
+  <xacro:plate num="1" parent="base_link"/>
   <xacro:mrobot_standoff_2in parent="standoff_2in_1_link" number="5" x_loc="0" y_loc="0" z_loc="${plate_height}"/>
   <xacro:mrobot_standoff_2in parent="standoff_2in_2_link" number="6" x_loc="0" y_loc="0" z_loc="${plate_height}"/>
   <xacro:mrobot_standoff_2in parent="standoff_2in_3_link" number="7" x_loc="0" y_loc="0" z_loc="${plate_height}"/>
   <xacro:mrobot_standoff_2in parent="standoff_2in_4_link" number="8" x_loc="0" y_loc="0" z_loc="${plate_height}"/>
-  <link name="plate_2_link">
-    <visual>
-      <geometry>
-        <cylinder radius="${base_link_radius}" length="${base_link_length}"/>
-      </geometry>
-      <origin xyz="0 0 0" rpy="0 0 0" />
-      <material name="yellow" />
-    </visual>
-    <collision>
-      <geometry>
-        <cylinder radius="${base_link_radius}" length="${base_link_length}"/>
-      </geometry>
-      <origin xyz="0 0 0" rpy="0 0 0" />
-    </collision>
-    <inertial>
-      <origin xyz="0 0 0" />
-      <mass value="0.1" />
-      <inertia ixx="0.01" ixy="0.0" ixz="0.0"
-               iyy="0.01" iyz="0.0"
-               izz="0.01" />
-    </inertial>
-  </link>
-  <joint name="plate_2_joint" type="fixed">
-    <origin xyz="0 0 ${plate_height}" rpy="0 0 0" />
-    <parent link="plate_1_link"/>
-    <child link="plate_2_link"/>
-  </joint>
+  <xacro:plate num="2" parent="plate_1_link"/>
 </robot>
