Commit message: Calculate inertia matrix using macro

File: mrobot_description/urdf/mrobot.urdf.xacro (robot description, xacro)
@@ -2,4 +2,5 @@
 <robot name="mrobot" xmlns:xacro="http://ros.org/wiki/xacro">
   <xacro:include filename="$(find mrobot_description)/urdf/common_properties.xacro"/>
+  <xacro:include filename="$(find mrobot_description)/urdf/inertia.urdf.xacro"/>
   <xacro:property name="wheel_radius" value="0.033"/>
   <xacro:property name="wheel_height" value="0.017"/>
@@ -33,8 +34,5 @@
     <inertial>
       <origin xyz="0 0 0" />
-      <mass value="2" />
-      <inertia ixx="0.001" ixy="0.0" ixz="0.0"
-               iyy="0.001" iyz="0.0"
-               izz="0.5" />
+      <xacro:cylinder_inertia m="${base_mass}" r="${base_link_radius}" h="${base_link_length}"/>
     </inertial>
   </link>
@@ -61,8 +59,5 @@
       <inertial>
         <origin xyz="0 0 0" />
-        <mass value="0.01" />
-        <inertia ixx="0.001" ixy="0.0" ixz="0.0"
-          iyy="0.001" iyz="0.0"
-          izz="0.001" />
+        <xacro:cylinder_inertia m="${wheel_mass}" r="${wheel_radius}" h="${wheel_height}"/>
       </inertial>
     </link>
@@ -93,8 +88,5 @@
       <inertial>
         <origin xyz="0 0 0" />
-        <mass value="0.001" />
-        <inertia ixx="0.0001" ixy="0.0" ixz="0.0"
-          iyy="0.0001" iyz="0.0"
-          izz="0.0001" />
+        <xacro:sphere_inertia m="${caster_mass}" r="${caster_radius}"/>
       </inertial>
     </link>
@@ -154,8 +146,5 @@
       <inertial>
         <origin xyz="0 0 0" />
-        <mass value="0.1" />
-        <inertia ixx="0.01" ixy="0.0" ixz="0.0"
-          iyy="0.01" iyz="0.0"
-          izz="0.01" />
+        <xacro:cylinder_inertia m="0.1" r="${base_link_radius}" h="${base_link_length}"/>
       </inertial>
     </link>

Commit message: Change the color of the wheels to black

File: mrobot_description/urdf/mrobot.urdf.xacro (robot description, xacro)
@@ -49,5 +49,5 @@
         </geometry>
         <origin xyz="0 0 0" rpy="${pi/2} 0 0"/>
-        <material name="white" />
+        <material name="black" />
       </visual>
       <collision>
